Commit message: Minimal pick-and-place using ros2 run jackal_ar4_goals pick_and_place X Y Z

File: src/ar4/ar4_description/urdf/ar4.urdf.xacro (robot description, xacro)
@@ -43,5 +43,5 @@
     <child link="link_2"/>
     <axis xyz="0 0 1"/>
-    <limit lower="${-42.0 / 180.0 * pi}" upper="${90.0 / 180.0 * pi}" effort="100" velocity="0.5"/>
+    <limit lower="${-42.0 / 180.0 * pi}" upper="${135.0 / 180.0 * pi}" effort="100" velocity="0.5"/>
   </joint>
   <xacro:link link_name="link_3"

File: src/ar4/ar4_description/urdf/gripper/ar_gripper_macro.xacro (robot description, xacro)
@@ -75,5 +75,22 @@
       <child link="${tf_prefix}gripper_jaw1_link"/>
       <axis xyz="-1 0 0"/>
-      <limit lower="0" upper="0.014" effort="-1" velocity="1.0"/>
+      <!-- effort must be positive (force limit in N). Original -1 caused Gazebo
+           to apply zero drive force, preventing the jaw from moving at all. -->
+      <!-- lower=-0.002: Gazebo spawns this joint at ~0 with floating-point noise
+           that can land at -9e-15 (slightly below 0).  A joint below its lower
+           limit triggers ODE's constraint enforcement, which fights the K_p
+           velocity drive even in the correct (opening) direction, permanently
+           locking the jaw.  Setting lower=-0.002 keeps the nominal closed
+           position (0.0 m) well above the hard stop so the constraint is
+           never active at spawn time.
+           upper=0.016: the K_p drive and arm-motion vibration can push the jaw
+           slightly past 0.014 after opening.  A jaw above its upper limit
+           triggers the same ODE constraint, locking jaw2 on the close stroke.
+           0.016 keeps the nominal open position (0.014 m) well below the hard
+           stop so the constraint never activates after an open command. -->
+      <limit lower="-0.002" upper="0.016" effort="20" velocity="1.0"/>
+      <!-- damping prevents oscillation across the 14 mm travel; friction holds
+           the jaw against whatever load is in the gripper at rest -->
+      <dynamics damping="0.1" friction="0.01"/>
     </joint>
     <joint name="${tf_prefix}gripper_jaw2_joint" type="prismatic">
@@ -82,6 +99,14 @@
       <child link="${tf_prefix}gripper_jaw2_link"/>
       <axis xyz="-1 0 0"/>
-      <limit lower="0" upper="0.014" effort="1000" velocity="1.0"/>
-      <mimic joint="${tf_prefix}gripper_jaw1_joint" multiplier="1" offset="0"/>
+      <!-- <mimic> removed: jaw2 is now an explicitly commanded joint via
+           ros2_control.  Keeping <mimic> while also registering a position
+           command interface causes GazeboSimSystem to fail initialisation
+           (ODE physics applies the mimic constraint AND ros2_control tries
+           to drive the joint independently, creating a conflict that prevents
+           any controllers — including joint_state_broadcaster — from loading,
+           which breaks the entire TF tree).  Joint state is published by
+           joint_state_broadcaster; robot_state_publisher picks it up normally. -->
+      <limit lower="-0.002" upper="0.016" effort="20" velocity="1.0"/>
+      <dynamics damping="0.1" friction="0.01"/>
     </joint>
   </xacro:macro>

File: src/clearpath_common/clearpath_platform_description/urdf/j100/j100.urdf.xacro (robot description, xacro)
@@ -32,8 +32,22 @@
         <material name="clearpath_dark_grey" />
       </visual>
+      <!-- Split the chassis collision into a lower body and a thin top plate.
+           The original single solid box (full chassis_height) blocked the arm
+           from planning to any pose below ar4_base_link because the box top
+           surface sits only ~10 mm below the arm mount.
+           The lower body covers the structural chassis (0 → 0.130 m).
+           The top plate (0.130 → 0.140 m) represents the deck surface.
+           The 44 mm gap above (0.140 → 0.184 m) is the open bay where the
+           arm mount passes through, freeing the planner for downward reaches. -->
       <collision>
-        <origin xyz="0 0 ${chassis_height/2}"/>
+        <origin xyz="0 0 0.065"/>
         <geometry>
-          <box size="${chassis_length} ${chassis_width} ${chassis_height}"/>
+          <box size="${chassis_length} ${chassis_width} 0.130"/>
+        </geometry>
+      </collision>
+      <collision>
+        <origin xyz="0 0 0.135"/>
+        <geometry>
+          <box size="${chassis_length} ${chassis_width} 0.010"/>
         </geometry>
       </collision>

File: src/jackal_ar4_description/urdf/ar4_arm.urdf.xacro (robot description, xacro)
@@ -29,5 +29,9 @@
       <child link="${prefix}link_1"/>
       <axis xyz="0 0 1"/>
-      <limit lower="${-170.0 / 180.0 * pi}" upper="${170.0 / 180.0 * pi}" effort="100" velocity="0.5"/>
+      <!-- velocity="2.0" > joint_limits.yaml max_velocity (1.0) so Gazebo never
+           caps below what MoveIt plans (0.8 * 1.0 = 0.8 rad/s) -->
+      <limit lower="${-170.0 / 180.0 * pi}" upper="${170.0 / 180.0 * pi}" effort="100" velocity="2.0"/>
+      <!-- damping: viscous drag kills overshoot; friction: static hold resists gravity at rest -->
+      <dynamics damping="0.1" friction="0.02"/>
     </joint>
     <xacro:link link_name="${prefix}link_2"
@@ -44,5 +48,9 @@
       <child link="${prefix}link_2"/>
       <axis xyz="0 0 1"/>
-      <limit lower="${-42.0 / 180.0 * pi}" upper="${90.0 / 180.0 * pi}" effort="100" velocity="0.5"/>
+      <limit lower="${-42.0 / 180.0 * pi}" upper="${135.0 / 180.0 * pi}" effort="100" velocity="2.0"/>
+      <!-- joint_2 (shoulder) carries the full arm weight ~1.1 kg at 0.3 m lever.
+           Damping must be high enough to resist gravity but not so high that the
+           joint can't track the MoveIt trajectory (which plans at 0.8 rad/s). -->
+      <dynamics damping="0.15" friction="0.05"/>
     </joint>
     <xacro:link link_name="${prefix}link_3"
@@ -59,5 +67,7 @@
       <child link="${prefix}link_3"/>
       <axis xyz="0 0 1"/>
-      <limit lower="${-89.0 / 180.0 * pi}" upper="${52.0 / 180.0 * pi}" effort="100" velocity="0.5"/>
+      <limit lower="${-89.0 / 180.0 * pi}" upper="${52.0 / 180.0 * pi}" effort="100" velocity="2.0"/>
+      <!-- joint_3 (elbow) carries links 3-6 ~0.65 kg; second most gravity-loaded joint -->
+      <dynamics damping="0.10" friction="0.03"/>
     </joint>
     <xacro:link link_name="${prefix}link_4"
@@ -74,5 +84,6 @@
       <child link="${prefix}link_4"/>
       <axis xyz="0 0 1"/>
-      <limit lower="${-1 * robot_parameters['j4_limit']}" upper="${robot_parameters['j4_limit']}" effort="100" velocity="0.5"/>
+      <limit lower="${-1 * robot_parameters['j4_limit']}" upper="${robot_parameters['j4_limit']}" effort="100" velocity="2.0"/>
+      <dynamics damping="0.05" friction="0.01"/>
     </joint>
     <xacro:link link_name="${prefix}link_5"
@@ -89,5 +100,6 @@
       <child link="${prefix}link_5"/>
       <axis xyz="0 0 1"/>
-      <limit lower="${-105.0 / 180.0 * pi}" upper="${105.0 / 180.0 * pi}" effort="100" velocity="1.0"/>
+      <limit lower="${-105.0 / 180.0 * pi}" upper="${105.0 / 180.0 * pi}" effort="100" velocity="3.0"/>
+      <dynamics damping="0.05" friction="0.01"/>
     </joint>
     <xacro:link link_name="${prefix}link_6"
@@ -104,5 +116,8 @@
       <child link="${prefix}link_6"/>
       <axis xyz="0 0 1"/>
-      <limit lower="${-1.0 * robot_parameters['j6_limit']}" upper="${robot_parameters['j6_limit']}" effort="100" velocity="1.0"/>
+      <limit lower="${-1.0 * robot_parameters['j6_limit']}" upper="${robot_parameters['j6_limit']}" effort="100" velocity="3.0"/>
+      <!-- joint_6 (wrist rotation) has been the main source of allowed_start_tolerance
+           violations — light damping reduces post-trajectory oscillation -->
+      <dynamics damping="0.05" friction="0.01"/>
     </joint>
     <xacro:include filename="$(find ar4_description)/urdf/gripper/ar_gripper_macro.xacro" />

File: src/jackal_ar4_description/urdf/jackal_ar4.ros2_control.xacro (robot description, xacro)
@@ -4,14 +4,36 @@
   <ros2_control name="JackalAR4Hardware" type="system">
     <hardware>
-      <plugin>mock_components/GenericSystem</plugin>
+      <!-- In simulation, GazeboSimSystem bridges ros2_control to Gazebo physics.
+           In real/RViz-only mode, mock_components echoes commands as states. -->
+      <xacro:if value="$(arg is_sim)">
+        <plugin>gz_ros2_control/GazeboSimSystem</plugin>
+        <!-- position_proportional_gain: GazeboSimSystem drives joints via
+             velocity = K_p * position_error.  Default K_p = 0.1 is far too
+             weak to resist gravity on the shoulder (joint_2) and elbow
+             (joint_3), causing the arm to fall after every trajectory.
+             2.0 is the empirically-determined maximum before instability. -->
+        <param name="position_proportional_gain">2.0</param>
+      </xacro:if>
+      <xacro:unless value="$(arg is_sim)">
+        <plugin>mock_components/GenericSystem</plugin>
+      </xacro:unless>
     </hardware>
-    <!-- AR4 Arm Joints (always present) -->
-    <joint name="ar4_joint_1"><command_interface name="position" /><state_interface name="position" /></joint>
-    <joint name="ar4_joint_2"><command_interface name="position" /><state_interface name="position" /></joint>
-    <joint name="ar4_joint_3"><command_interface name="position" /><state_interface name="position" /></joint>
-    <joint name="ar4_joint_4"><command_interface name="position" /><state_interface name="position" /></joint>
-    <joint name="ar4_joint_5"><command_interface name="position" /><state_interface name="position" /></joint>
-    <joint name="ar4_joint_6"><command_interface name="position" /><state_interface name="position" /></joint>
-    <joint name="ar4_gripper_jaw1_joint"><command_interface name="position" /><state_interface name="position" /></joint>
+    <!-- AR4 Arm Joints (always present)
+         velocity state_interface is required for the JointTrajectoryController
+         to properly track trajectories and hold position between moves.
+         Without it the JTC has no velocity feedback, causing the arm to drift
+         under gravity when it transitions between trajectory segments. -->
+    <joint name="ar4_joint_1"><command_interface name="position" /><state_interface name="position" /><state_interface name="velocity" /></joint>
+    <joint name="ar4_joint_2"><command_interface name="position" /><state_interface name="position" /><state_interface name="velocity" /></joint>
+    <joint name="ar4_joint_3"><command_interface name="position" /><state_interface name="position" /><state_interface name="velocity" /></joint>
+    <joint name="ar4_joint_4"><command_interface name="position" /><state_interface name="position" /><state_interface name="velocity" /></joint>
+    <joint name="ar4_joint_5"><command_interface name="position" /><state_interface name="position" /><state_interface name="velocity" /></joint>
+    <joint name="ar4_joint_6"><command_interface name="position" /><state_interface name="position" /><state_interface name="velocity" /></joint>
+    <!-- Gripper jaws: in the same GazeboSimSystem instance as the arm to avoid
+         joint ownership races.  Two separate plugin instances on the same model
+         scan all joints non-deterministically; merging prevents one instance from
+         "stealing" jaw commands intended for the other. -->
+    <joint name="ar4_gripper_jaw1_joint"><command_interface name="position" /><state_interface name="position" /><state_interface name="velocity" /></joint>
+    <joint name="ar4_gripper_jaw2_joint"><command_interface name="position" /><state_interface name="position" /><state_interface name="velocity" /></joint>
     <!--
       Wheel joints: excluded in sim because Gazebo diff_drive owns them.

File: src/jackal_ar4_description/urdf/jackal_ar4.urdf (robot description, URDF)
Before this commit: robot jackal_ar4, 19 links, 18 joints
Joints:
- joint ar4_joint_2: limit lower=-0.7330382858376184 upper=1.5707963267948966 effort=100 velocity=0.5 -> lower=-0.7330382858376184 upper=2.3561944901923448 effort=100 velocity=0.5

File: src/jackal_ar4_description/urdf/jackal_ar4.urdf.xacro (robot description, xacro)
@@ -4,4 +4,8 @@
   <xacro:arg name="arm_prefix" default="ar4_" />
   <xacro:arg name="is_sim" default="false" />
+  <!-- Path to ros2_controllers.yaml consumed by the gz_ros2_control Gazebo plugin -->
+  <xacro:arg name="gazebo_controllers"
+    default="$(find jackal_ar4_moveit_config)/config/ros2_controllers.yaml" />
+  <xacro:arg name="namespace" default="" />
   <!-- Include Common Materials and macros -->
   <xacro:include filename="$(find clearpath_platform_description)/urdf/common.urdf.xacro" />
@@ -90,4 +94,18 @@
       </plugin>
     </gazebo>
+    <!-- gz_ros2_control: hosts the controller_manager inside Gazebo and wires
+         ros2_control hardware interfaces to Gazebo joint physics.
+         This replaces the standalone ros2_control_node in the launch. -->
+    <gazebo>
+      <plugin filename="libgz_ros2_control-system.so"
+              name="gz_ros2_control::GazeboSimROS2ControlPlugin">
+        <parameters>$(arg gazebo_controllers)</parameters>
+        <ros>
+          <namespace>$(arg namespace)</namespace>
+          <remapping>/tf:=tf</remapping>
+          <remapping>/tf_static:=tf_static</remapping>
+        </ros>
+      </plugin>
+    </gazebo>
   </xacro:if>
 </robot>
