Commit message: Add LiDAR support and A* navigation launch files for Jackal AR4
- Introduced LiDAR link and joint in URDF for accurate sensor representation.
- Updated costmap parameters to include obstacle layer using LiDAR data.
- Created astar_navigation.launch.py for A* planner integration with Gazebo.
- Added mapping.launch.py for SLAM Toolbox mapping sessions.
- Implemented twist_unstamper.py to convert TwistStamped to Twist for compatibility.

File: src/jackal_ar4_description/urdf/jackal_ar4.urdf.xacro (robot description, xacro)
@@ -63,4 +63,29 @@
   <!-- ros2_control -->
   <xacro:include filename="$(find jackal_ar4_description)/urdf/jackal_ar4.ros2_control.xacro" />
+  <!-- ── LiDAR link (always present so TF tree is complete) ──────────────
+       Mounted at front-centre of chassis, 15 cm above chassis_link.
+       Named 'lidar' to match mobo_bot sensor reference convention.
+  -->
+  <link name="lidar">
+    <visual>
+      <origin xyz="0 0 -0.02"/>
+      <geometry><cylinder radius="0.03" length="0.04"/></geometry>
+      <material name="clearpath_black"/>
+    </visual>
+    <collision>
+      <origin xyz="0 0 -0.02"/>
+      <geometry><cylinder radius="0.03" length="0.04"/></geometry>
+    </collision>
+    <inertial>
+      <mass value="0.2"/>
+      <origin xyz="0 0 -0.02" rpy="0 0 0"/>
+      <inertia ixx="0.0001" ixy="0" ixz="0" iyy="0.0001" iyz="0" izz="0.0001"/>
+    </inertial>
+  </link>
+  <joint name="lidar_joint" type="fixed">
+    <parent link="chassis_link"/>
+    <child link="lidar"/>
+    <origin xyz="0.18 0.0 0.15" rpy="0 0 0"/>
+  </joint>
   <!-- ── Gazebo plugins (only when is_sim:=true) ──────────────────────── -->
   <xacro:if value="$(arg is_sim)">
@@ -108,4 +133,36 @@
       </plugin>
     </gazebo>
+    <!-- LiDAR sensor: 360° 10Hz gpu_lidar, topic: lidar/scan
+         Pattern follows mobo_bot robot_gazebo_properties.xacro exactly.
+         gz_frame_id must match link name for RViz LaserScan display. -->
+    <gazebo reference="lidar">
+      <sensor name="lidar" type="gpu_lidar">
+        <topic>lidar/scan</topic>
+        <gz_frame_id>lidar</gz_frame_id>
+        <always_on>true</always_on>
+        <visualize>true</visualize>
+        <update_rate>10.0</update_rate>
+        <ray>
+          <scan>
+            <horizontal>
+              <samples>360</samples>
+              <min_angle>-3.14159265</min_angle>
+              <max_angle>3.14159265</max_angle>
+              <resolution>1</resolution>
+            </horizontal>
+          </scan>
+          <range>
+            <min>0.12</min>
+            <max>12.0</max>
+            <resolution>0.01</resolution>
+          </range>
+          <noise>
+            <type>gaussian</type>
+            <mean>0.0</mean>
+            <stddev>0.01</stddev>
+          </noise>
+        </ray>
+      </sensor>
+    </gazebo>
   </xacro:if>
 </robot>

Commit message: Fix mission executive: workspace model and navigation precision
  - Increase workspace_radius to 0.15m for navigation tolerance
  - Tighten arrival_threshold to 0.20m for precise goal arrival
  - Fix debounce to only apply during NAVIGATING state
  - Add ROTATING, SETTLING, FINE_APPROACH states
  - Add nav timeout and idle timeout
  - Update bottle pick height to 0.115m
  - Add all-in-one bringup launch file

File: src/jackal_ar4_description/urdf/jackal_ar4.urdf.xacro (robot description, xacro)
@@ -90,5 +90,7 @@
   <!-- ── Gazebo plugins (only when is_sim:=true) ──────────────────────── -->
   <xacro:if value="$(arg is_sim)">
-    <!-- Differential drive: wheels physics + /odom + /tf odom->base_link -->
+    <!-- Differential drive: wheels physics + /odom + /tf odom->base_link.
+         Odom drifts over time due to wheel slip; AMCL corrects the drift
+         by publishing map->odom from LiDAR-to-map matching. -->
     <gazebo>
       <plugin filename="gz-sim-diff-drive-system"
@@ -131,4 +133,18 @@
           <remapping>/tf_static:=tf_static</remapping>
         </ros>
+      </plugin>
+    </gazebo>
+    <!-- Ground-truth odometry from physics engine (no wheel drift).
+         Publishes gz.msgs.Odometry on /ground_truth_odom at 10 Hz.
+         Bridged to ROS by gazebo.launch.py, consumed by gz_ground_truth_odom.py
+         to compute map→odom correction. No subprocess, no performance hit. -->
+    <gazebo>
+      <plugin filename="gz-sim-odometry-publisher-system"
+              name="gz::sim::systems::OdometryPublisher">
+        <odom_topic>ground_truth_odom</odom_topic>
+        <odom_frame>map</odom_frame>
+        <robot_base_frame>base_link</robot_base_frame>
+        <odom_publish_frequency>10</odom_publish_frequency>
+        <dimensions>3</dimensions>
       </plugin>
     </gazebo>
@@ -165,4 +181,31 @@
       </sensor>
     </gazebo>
+    <!-- Collision bitmask: robot=0x01, bottles=0x02.
+         0x01 & 0x02 == 0 → robot links pass through bottles.
+         Robot still collides with ground/walls/table (default 0xFFFF). -->
+    <xacro:macro name="no_bottle_collision" params="link_name">
+      <gazebo reference="${link_name}">
+        <collision><surface><contact>
+          <collide_bitmask>0x01</collide_bitmask>
+        </contact></surface></collision>
+      </gazebo>
+    </xacro:macro>
+    <xacro:no_bottle_collision link_name="chassis_link"/>
+    <xacro:no_bottle_collision link_name="front_left_wheel_link"/>
+    <xacro:no_bottle_collision link_name="front_right_wheel_link"/>
+    <xacro:no_bottle_collision link_name="rear_left_wheel_link"/>
+    <xacro:no_bottle_collision link_name="rear_right_wheel_link"/>
+    <xacro:no_bottle_collision link_name="ar4_mount_plate"/>
+    <xacro:no_bottle_collision link_name="lidar"/>
+    <xacro:no_bottle_collision link_name="ar4_base_link"/>
+    <xacro:no_bottle_collision link_name="ar4_link_1"/>
+    <xacro:no_bottle_collision link_name="ar4_link_2"/>
+    <xacro:no_bottle_collision link_name="ar4_link_3"/>
+    <xacro:no_bottle_collision link_name="ar4_link_4"/>
+    <xacro:no_bottle_collision link_name="ar4_link_5"/>
+    <xacro:no_bottle_collision link_name="ar4_link_6"/>
+    <xacro:no_bottle_collision link_name="ar4_gripper_base_link"/>
+    <xacro:no_bottle_collision link_name="ar4_gripper_jaw1_link"/>
+    <xacro:no_bottle_collision link_name="ar4_gripper_jaw2_link"/>
   </xacro:if>
 </robot>
